File: hapia (1).kicad_sch (KiCad schematic)
At the start: 192 parts, among them J1 Micro_SD_Card, J10 USB_C_Receptacle_USB2.0_16P, J11 USB_A, J12 Micro_SD_Card, J2 SUB_placa_de_controle, J3 Conn_01x15_Pin, J4 ATX-20, J5 Conn_01x10, J6 Conn_01x04_Pin, J7 Conn_01x04_Pin, J8 Conn_01x04_Pin, J9 Conn_01x04_Pin, M1 Fan, M2 Fan, M3 Fan, Q1 NMOS, Q2 NMOS, Q3 NMOS, Q4 NMOS, SW1 SW_Push, SW2 SW_Push, U1 SRV05-4, U10 SRV05-4, U2 STM32F407VETx, U3 TMC2209-LA, U4 TMC2209-LA, U5 TPS54302, U6 TMC2209-LA, U7 TMC2209-LA, U8 MIC4427, U9 MIC4427, Y1 Crystal

Commit message: Add files via upload
V0,5
Parts:
- removed C71, C79: 100nf, symbol Device:C
- removed J11: USB_A, Connector_USB:USB_A_Molex_67643_Horizontal, symbol Connector:USB_A
- removed J12: Micro_SD_Card, symbol Connector:Micro_SD_Card
- removed J5: Conn_01x10, symbol Connector_Generic:Conn_01x10
- removed M1, M3: Fan, symbol Motor:Fan
- removed Q3, Q4: NMOS, symbol Simulation_SPICE:NMOS
- removed R25, R5: 33r, symbol Device:R
- removed RN1, RN2: 33Ω, Resistor_SMD:R_Array_Convex_8x0602, symbol Device:R_Pack08_Split
- removed U9: MIC4427, symbol Driver_FET:MIC4427
- added C27, C74: 10nf, symbol Device:C
- added C53, C75: 100nf, symbol Device:C
- added C59: 4.7uf, symbol Device:C
- added C62: 1uf, symbol Device:C
- added D1: D_Schottky, symbol Device:D_Schottky
- added J10: Conn_01x20, symbol Connector_Generic:Conn_01x20
- added J11: Conn_01x10, symbol Connector_Generic:Conn_01x10
- added J12, J13, J14: Conn_01x03, symbol Connector_Generic:Conn_01x03
- added J16: Conn_01x07, symbol Connector_Generic:Conn_01x07
- added R46, R47, R48, R49, R50, R51, R52, R53, R62, R63, R64, R65, R66, R67, R69, R70, R71, R72, R79, R80, R81: 33r, symbol Device:R
- added R82, R85, R87: 10kΩ, symbol Device:R
- added R83, R84, R86, R88: 1kΩ, symbol Device:R
- added U10, U9: SRV05-4, Package_TO_SOT_SMD:SOT-23-6, symbol Power_Protection:SRV05-4
- C3: renamed from C13; value pf -> 22pf; footprint (none) -> Capacitor_SMD:C_0603_1608Metric; ID: (none) -> C1653
- C4: renamed from C1; value pf -> 22pf; footprint (none) -> Capacitor_SMD:C_0603_1608Metric; ID: (none) -> C1653
- C52: renamed from C51; value 470uf -> 1000uf
- C55: renamed from C54; value 100µf -> 1000µf
- C60: renamed from C23; value 470µf -> 1000uf
- J2: renamed from J1; footprint (none) -> Connector_Card:microSD_HC_Molex_104031-0811; ID: (none) -> C585350
- R68, R73: value 10k -> 33r
- R74, R75: value R -> 33r
- R78: value 1kΩ -> 33r
- Y1: value Crystal -> 8mhz; footprint (none) -> Crystal:Crystal_SMD_Abracon_ABM7-2Pin_6.0x3.5mm; ID: (none) -> C5564812
- renumbered C17 to C1, C52 to C10, C27 to C11, C30 to C12, C34 to C13, C33 to C14, C38 to C15, C46 to C16, C28 to C17, C47 to C18, C50 to C19, C14 to C2, C39 to C20, C44 to C21, C43 to C22, C31 to C23, C32 to C24, C35 to C25, C36 to C26, C42 to C28, C41 to C29, C45 to C30, C48 to C31, C56 to C32, C57 to C33, C58 to C34, C59 to C35, C61 to C36, C62 to C37, C63 to C38, C64 to C39, C65 to C40, C66 to C41, C67 to C42, C68 to C43, C69 to C44, C70 to C45, C72 to C46, C73 to C47, C74 to C48, C75 to C49, C3 to C5, C76 to C50, C77 to C51, C60 to C54, C18 to C56, C19 to C57, C20 to C58, C2 to C6, C21 to C61, C4 to C63, C5 to C64, C6 to C65, C7 to C66, C8 to C67, C9 to C68, C10 to C69, C40 to C7, C11 to C70, C15 to C71, C12 to C72, C16 to C73, C29 to C76, C37 to C77, C26 to C8, C49 to C9, D1 to D2, D2 to D3, F3 to F1, F4 to F3, F1 to F4, FB2 to FB1, FB1 to FB2, J4 to J1, J7 to J3, J6 to J4, J8 to J5, J9 to J6, J3 to J7, J2 to J8, J10 to J9, M2 to M1, Q1 to Q2, Q2 to Q3, R2 to R1, R42 to R10, R44 to R11, R41 to R12, R43 to R13, R45 to R14, R47 to R15, R49 to R16, R55 to R17, R56 to R18, R57 to R19, R1 to R2, R58 to R20, R59 to R21, R60 to R22, R61 to R23, R62 to R24, R63 to R25, R64 to R26, R34 to R27, R38 to R28, R35 to R29, R53 to R3, R39 to R30, R36 to R31, R40 to R32, R30 to R33, R31 to R34, R32 to R35, R22 to R36, R65 to R37, R71 to R38, R66 to R39, R54 to R4, R67 to R40, R70 to R41, R4 to R42, R28 to R43, R3 to R44, R29 to R45, R48 to R5, R26 to R54, R27 to R55, R69 to R56, R23 to R57, R24 to R58, R72 to R59, R50 to R6, R51 to R60, R52 to R61, R33 to R7, R37 to R8, R46 to R9, SW2 to SW1, SW1 to SW2, TP5 to TP1, TP7 to TP3, TP6 to TP4, TP1 to TP5, TP3 to TP6, TP4 to TP7, U2 to U1, U8 to U13, U4 to U2, U5 to U3, U3 to U4, U6 to U5, U7 to U6, U10 to U7, U1 to U8
Connections:
- net Fan_1_D is gone; now on an unnamed net: R68.1
- net Fan_2_D is gone; now on an unnamed net: R73.1
- net +12V: now also C53.2, C59.1, C75.1, J11.4 (Pin_4), J11.6 (Pin_6)
- net +3.3V: now also C27.2, D1.2 (A), J10.19 (Pin_19), J10.20 (Pin_20), J11.1 (Pin_1), J11.2 (Pin_2), J11.3 (Pin_3), R82.1, R85.1, R87.1, R88.2, U10.2 (VN), U10.6 (IO4), U9.2 (VN)
- net +5V: now also J11.5 (Pin_5), J11.7 (Pin_7)
- net GND: now also C13.1, C14.1, C15.1, C16.1, C18.1, C19.1, C20.1, C21.1, C22.1, C23.1, C24.1, C25.1, C26.1, C28.1, C29.1, C30.1, C31.1, C34.1, C35.1, C36.1, C37.1, C38.1, C39.1, C40.1, C41.1, C42.1, C43.1, C44.1, C45.1, C46.1, C47.1, C48.1, C49.1, C50.1, C51.1, C52.1, C55.2, C78.2, M1.2 (-), Q2.3 (S), Q3.3 (S), R10.1, R11.1, R18.1, R20.1, R23.2, R24.2, R25.2, R26.2, R39.2, R40.2, R5.2, R6.2, U13.3 (GND), U2.18 (GND), U2.20 (STDBY), U2.29 (GND), U2.3 (GND), U4.20 (STDBY), U5.18 (GND), U5.20 (STDBY), U5.29 (GND), U5.3 (GND), U6.18 (GND), U6.20 (STDBY), U6.29 (GND), U6.3 (GND), C27.1, C53.1, C59.2, C62.2, C74.2, C75.2, J11.10 (Pin_10), J11.8 (Pin_8), J11.9 (Pin_9), J12.3 (Pin_3), J13.3 (Pin_3), J14.3 (Pin_3), J16.1 (Pin_1), J16.7 (Pin_7), U10.5 (VP), U9.5 (VP); no longer R75.2
- net SUB_1: now also U1.92 (PB6)
- net SUB_2: now also U1.93 (PB7); no longer U1.91 (PB5)
- net SUB_3: now also U1.95 (PB8); no longer U1.92 (PB6)
- net SUB_4: now also U1.96 (PB9); no longer U1.93 (PB7)
- net SUB_5: now also U1.97 (PE0); no longer U1.95 (PB8)
- net SUB_6: now also U1.98 (PE1); no longer U1.96 (PB9)
- net exrtusora_d: no longer Q3.2 (G), R40.1
- net at U1.82 (PD1): now also R52.1
- net at U1.81 (PD0): now also R53.1
- net at U1.86 (PD5): now also R48.1
- net at U1.58 (PD11): now also R65.1
- net at U1.55 (PD8): now also R62.1
- net at R78.1: now also U1.45 (PE14); no longer U1.65 (PC8)
- net at C61.1, FB2.1, TP1.1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: now also C62.1, C74.1
- net at U1.43 (PE12): now also R77.1
- net at U1.44 (PE13): now also R70.1
- net at U1.46 (PE15): now also R79.1
- net at U1.47 (PB10): now also R76.1
- net at U1.48 (PB11): now also R75.1
- net at U1.51 (PB12): now also R74.1
- net at U1.53 (PB14): now also R72.1
- net at U1.54 (PB15): now also R71.1
- net at U1.56 (PD9): now also R63.1
- net at U1.57 (PD10): now also R64.1
- net at U1.59 (PD12): now also R66.1
- net at U1.60 (PD13): now also R67.1
- net at U1.62 (PD15): now also R69.1
- net at U1.63 (PC6): no longer R77.1
- net at U1.64 (PC7): no longer R76.1
- net SEN_3: now reaches U1.69 (PA10)
- net SEN_3: now also R86.1, U9.4 (IO3)
- net SEN_2: now reaches U1.70 (PA11)
- net SEN_2: now also R84.1, U9.3 (IO2)
- net SEN_1: now reaches U1.71 (PA12)
- net SEN_1: now also R83.1, U9.1 (IO1)
- net at U1.72 (PA13): now also R81.1
- net at U1.76 (PA14): now also R80.1
- net at U1.83 (PD2): now also R51.1
- net at U1.84 (PD3): now also R50.1
- net at U1.85 (PD4): now also R49.1
- net at U1.87 (PD6): now also R47.1
- net at U1.88 (PD7): now also R46.1
- net at R54.1: now also U1.90 (PB4); no longer U1.89 (PB3)
- net at R55.1: now also U1.91 (PB5); no longer U1.90 (PB4)
- removed net PGND: C13.1, C14.1, C15.1, C16.1, C18.1, C19.1, C20.1, C21.1, C22.1, C23.1, C24.1, C25.1, C26.1, C28.1, C29.1, C30.1, C31.1, C34.1, C35.1, C36.1, C37.1, C38.1, C39.1, C40.1, C41.1, C42.1, C43.1, C44.1, C45.1, C46.1, C47.1, C48.1, C49.1, C50.1, C51.1, C52.1, C55.2, C78.2, M1.2 (-), Q2.3 (S), R10.1, R11.1, R18.1, R20.1, R23.2, R24.2, R25.2, R26.2, R39.2, R40.2, R5.2, R6.2, R68.2, R73.2, U13.3 (GND), U2.18 (GND), U2.20 (STDBY), U2.29 (GND), U2.3 (GND), U4.20 (STDBY), U5.18 (GND), U5.20 (STDBY), U5.29 (GND), U5.3 (GND), U6.18 (GND), U6.20 (STDBY), U6.29 (GND), U6.3 (GND)
- net STM_ADC renamed gpi_PA_13
- net STM_ADC_1 renamed gpi_PA_14
- net USB_det: no longer names the net of J9.A4 (VBUS), J9.A9 (VBUS), J9.B4 (VBUS), J9.B9 (VBUS), TP10.1, U7.2 (VN)
- net USB_det: no longer R74.1
- removed net USB_det_2.5v: R74.2, R75.1, R78.2
- net gpi_PD0 renamed gpi_pd_0
- net gpi_pd_0: now also R53.2
- net gpi_PD1 renamed gpi_pd_1
- net gpi_pd_1: now also R52.2
- net gpi_PD14 renamed gpi_PB_10
- net gpi_PB_10: now also J10.14 (Pin_14)
- net gpi_PD15 renamed gpi_PE_12
- net gpi_PE_12: now also J10.15 (Pin_15)
- net gpi_PD2 renamed gpi_pd_2
- net gpi_pd_2: now also R51.2
- net gpi_PD3 renamed gpi_pd_3
- net gpi_pd_3: now also R50.2
- net gpi_PD4 renamed gpi_pd_4
- net gpi_pd_4: now also R49.2
- net gpi_PD5 renamed gpi_pd_5
- net gpi_pd_5: now also R48.2
- net gpi_PD6 renamed gpi_pd_6
- net gpi_pd_6: now also R47.2
- net gpi_PD7 renamed gpi_pd_7
- net gpi_pd_7: now also R46.2
- new net: J12.1 (Pin_1), R82.2
- new net: D1.1 (K), J16.6 (Pin_6)
- new net: J13.1 (Pin_1), R85.2
- new net: J13.2 (Pin_2), R84.2
- new net: J16.5 (Pin_5), R88.1
- new net: J14.1 (Pin_1), R87.2
- new net: J14.2 (Pin_2), R86.2
- new net: J12.2 (Pin_2), R83.2
- new net SW0: J16.4 (Pin_4), U1.89 (PB3), U10.4 (IO3)
- new net SWCLK: J16.3 (Pin_3), R80.2, U10.3 (IO2)
- new net SWDIO: J16.2 (Pin_2), R81.2, U10.1 (IO1)
- new net exrtusora_s: Q3.2 (G), R40.1
- new net gpi_PB_11: J10.13 (Pin_13), R75.2
- new net gpi_PB_12: J10.12 (Pin_12), R74.2
- new net gpi_PB_13: J10.11 (Pin_11), R73.2
- new net gpi_PB_14: J10.10 (Pin_10), R72.2
- new net gpi_PB_15: J10.9 (Pin_9), R71.2
- new net gpi_PE_13: J10.16 (Pin_16), R70.2
- new net gpi_PE_14: J10.17 (Pin_17), R78.2
- new net gpi_PE_15: J10.18 (Pin_18), R79.2
- new net gpi_pd_10: J10.3 (Pin_3), R64.2
- new net gpi_pd_11: J10.4 (Pin_4), R65.2
- new net gpi_pd_12: J10.5 (Pin_5), R66.2
- new net gpi_pd_13: J10.6 (Pin_6), R67.2
- new net gpi_pd_14: J10.7 (Pin_7), R68.2
- new net gpi_pd_15: J10.8 (Pin_8), R69.2
- new net gpi_pd_8: J10.1 (Pin_1), R62.2
- new net gpi_pd_9: J10.2 (Pin_2), R63.2
- no-connect marks 76 -> 38
Other:
- moved on the sheet: C29, C60, C61, C76, C77, D2, FB2, M1, R54, R55, R60, R61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
