File: d-nmos.kicad_sch (KiCad schematic)
At the start: 7 parts, among them Q13 PMOS, Q26 NMOS

Commit message: 21082026/G
falta muita coisa
Parts:
- renumbered C59 to C95, Q26 to Q10, Q13 to Q9, R114 to R108, R115 to R109, R116 to R110, R117 to R111
