File: potencia_misc.kicad_sch (KiCad schematic)
At the start: 60 parts, among them J7 ATX-24, M1 Fan, M2 Fan, M3 Fan, Q4 NMOS, Q5 NMOS, SW3 SW_Push, U11 UCC27524DR, U12 UCC27524DR, U13 IRFS7530TRL7PP, U14 IRFS7530TRL7PP, U8 TPS62933F

Commit message: 05092026/00001
Parts:
- removed SW3: SW_Push, Connector_PinHeader_2.54mm:PinHeader_1x02_P2.54mm_Vertical, symbol Switch:SW_Push
- removed TP13: TestPoint, TestPoint:TestPoint_Pad_D1.0mm, symbol Connector:TestPoint
- removed U11, U12: UCC27524DR, Package_SO:SOIC-8_3.9x4.9mm_P1.27mm, symbol Driver_FET:UCC27524D
- added R118, R119: 12Ω, Resistor_SMD:R_MELF_MMB-0207, symbol Device:R
- added TP17: -12v, TestPoint:TestPoint_Pad_D1.0mm, symbol Connector:TestPoint
- added TP18: atx3.3v, TestPoint:TestPoint_Pad_D1.0mm, symbol Connector:TestPoint
- added U15, U16, U17, U18: UCC27517DBVR, Package_TO_SOT_SMD:SOT-23-5, symbol FET_driver_p:UCC27517DBVR
- R73: value 10kΩ -> 2.2kΩ; footprint (none) -> Resistor_SMD:R_0603_1608Metric Resistor_SMD:R_0603_1608Metric; jlc_pcb: (none) -> C13564; mouser: (none) -> 81-NCP18XH103F03RB; mpn (none) -> NCP18XH103F03RB
- R74: value 10kΩ -> 1.2kΩ; footprint (none) -> Resistor_SMD:R_0603_1608Metric Resistor_SMD:R_0603_1608Metric; jlc_pcb: (none) -> C13564; mouser: (none) -> 81-NCP18XH103F03RB; mpn (none) -> NCP18XH103F03RB
- R78, R79, R80, R81, R82: footprint (none) -> Resistor_SMD:R_0603_1608Metric Resistor_SMD:R_0603_1608Metric; jlc_pcb: (none) -> C13564; mouser: (none) -> 81-NCP18XH103F03RB; mpn (none) -> NCP18XH103F03RB
Connections:
- net +3.3V: now also U15.1 (VCC), U16.1 (VCC), U17.1 (VCC), U18.1 (VCC)
- net Fan_1: now also U15.3 (IN_+)
- net Fan_2: now also U16.3 (IN_+)
- net GND: now also U15.2 (GND), U15.4 (IN_-), U16.2 (GND), U16.4 (IN_-), U17.2 (GND), U17.4 (IN_-), U18.2 (GND), U18.4 (IN_-)
- net exrtusora: now also U17.3 (IN_+)
- net hot_bed: now also U18.3 (IN_+)
- net at R109.1: now also U17.5 (OUT)
- net at R108.1: now also R79.1, U13.1 (G)
- net at Q5.2 (G), R82.1: now also R119.2
- net at Q4.2 (G), R81.1: now also R118.2
- net at J7.1 (+3.3V), J7.12 (+3.3V), J7.13 (+3.3V)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: now also TP18.1
- net at J7.14 (-12V): now also TP17.1
- new net: R108.2, U18.5 (OUT)
- new net: R118.1, U15.5 (OUT)
- new net: R119.1, U16.5 (OUT)
- no-connect marks 2 -> 0
Other:
- moved on the sheet: R108, R81, R82

Commit message: 27092026/0002
Parts:
- Q4, Q5: value NMOS -> IRFL4315TRPBF; footprint (none) -> Package_TO_SOT_SMD:SOT-223-3_TabPin2; jlc_pcb: (none) -> C537930; mouser: (none) -> 942-IRFL4315TRPBF; mpn (none) -> IRFL4315TRPBF
- R73, R74, R78, R79, R80, R81, R82: footprint Resistor_SMD:R_0603_1608Metric Resistor_SMD:R_0603_1608Metric -> Resistor_SMD:R_0603_1608Metric Resistor_SMD_R_0603_1608Metric
Changed lines of the file:
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@@
 			)
 		)
-		(property "Footprint" "Resistor_SMD:R_0603_1608Metric Resistor_SMD:R_0603_1608Metric"
+		(property "Footprint" "Resistor_SMD:R_0603_1608Metric Resistor_SMD_R_0603_1608Metric"
 			(at 256.032 52.07 90)
 			(hide yes)
@@
 			)
 		)
-		(property "Value" "NMOS"
+		(property "Value" "IRFL4315TRPBF"
 			(at 279.4 123.1899 0)
 			(show_name no)
@@
 			)
 		)
-		(property "Footprint" ""
+		(property "Footprint" "Package_TO_SOT_SMD:SOT-223-3_TabPin2"
 			(at 278.13 119.38 0)
 			(hide yes)
@@
 			)
 		)
-		(property "Datasheet" "https://ngspice.sourceforge.io/docs/ngspice-html-manual/manual.xhtml#cha_MOSFETs"
+		(property "Datasheet" "https://www.lcsc.com/datasheet/C537930.pdf?spm=wm.sxq.inf.ggs___wm.fly.bg.10.xh&lcsc_vid=TgUMVVJTT1APU1ICElJZUAAEEgNaVFJfFlJeUQADFVYxVlNeT1ZfVlJXQ1lcUzsOAxUeFF5JWBYZEEoKFBINSQcJGk4NBhADEA4cHktXQ1JYSQwSGg0%3D"
 			(at 273.05 134.62 0)
 			(hide yes)
@@
 			)
 		)
+		(property "jlc_pcb:" "C537930"
+			(at 273.05 121.92 0)
+			(hide yes)
+			(show_name no)
+			(do_not_autoplace no)
+			(effects
+				(font
+					(size 1.27 1.27)
+				)
+			)
+		)
+		(property "mpn" "IRFL4315TRPBF"
+			(at 273.05 121.92 0)
+			(hide yes)
+			(show_name no)
+			(do_not_autoplace no)
+			(effects
+				(font
+					(size 1.27 1.27)
+				)
+			)
+		)
+		(property "mouser:" "942-IRFL4315TRPBF"
+			(at 273.05 121.92 0)
+			(hide yes)
+			(show_name no)
+			(do_not_autoplace no)
+			(effects
+				(font
+					(size 1.27 1.27)
+				)
+			)
+		)
+		(property "Descrição" ""
+			(at 273.05 121.92 0)
+			(hide yes)
+			(show_name no)
+			(do_not_autoplace no)
+			(effects
+				(font
+					(size 1.27 1.27)
+				)
+			)
+		)
 		(pin "1"
 		)
@@
 			)
 		)
-		(property "Footprint" "Resistor_SMD:R_0603_1608Metric Resistor_SMD:R_0603_1608Metric"
+		(property "Footprint" "Resistor_SMD:R_0603_1608Metric Resistor_SMD_R_0603_1608Metric"
 			(at 44.958 217.805 90)
 			(hide yes)
@@
 			)
 		)
-		(property "Footprint" "Resistor_SMD:R_0603_1608Metric Resistor_SMD:R_0603_1608Metric"
+		(property "Footprint" "Resistor_SMD:R_0603_1608Metric Resistor_SMD_R_0603_1608Metric"
 			(at 44.958 210.185 90)
 			(hide yes)
@@
 			)
 		)
-		(property "Value" "NMOS"
+		(property "Value" "IRFL4315TRPBF"
 			(at 279.4 160.0199 0)
 			(show_name no)
@@
 			)
 		)
-		(property "Footprint" ""
+		(property "Footprint" "Package_TO_SOT_SMD:SOT-223-3_TabPin2"
 			(at 278.13 156.21 0)
 			(hide yes)
@@
 			)
 		)
-		(property "Datasheet" "https://ngspice.sourceforge.io/docs/ngspice-html-manual/manual.xhtml#cha_MOSFETs"
+		(property "Datasheet" "https://www.lcsc.com/datasheet/C537930.pdf?spm=wm.sxq.inf.ggs___wm.fly.bg.10.xh&lcsc_vid=TgUMVVJTT1APU1ICElJZUAAEEgNaVFJfFlJeUQADFVYxVlNeT1ZfVlJXQ1lcUzsOAxUeFF5JWBYZEEoKFBINSQcJGk4NBhADEA4cHktXQ1JYSQwSGg0%3D"
 			(at 273.05 171.45 0)
 			(hide yes)
@@
 			)
 		)
+		(property "jlc_pcb:" "C537930"
+			(at 273.05 158.75 0)
+			(hide yes)
+			(show_name no)
+			(do_not_autoplace no)
+			(effects
+				(font
+					(size 1.27 1.27)
+				)
+			)
+		)
+		(property "mouser:" "942-IRFL4315TRPBF"
+			(at 273.05 158.75 0)
+			(hide yes)
+			(show_name no)
+			(do_not_autoplace no)
+			(effects
+				(font
+					(size 1.27 1.27)
+				)
+			)
+		)
+		(property "mpn" "IRFL4315TRPBF"
+			(at 273.05 158.75 0)
+			(hide yes)
+			(show_name no)
+			(do_not_autoplace no)
+			(effects
+				(font
+					(size 1.27 1.27)
+				)
+			)
+		)
 		(pin "1"
 		)
@@
 			)
 		)
-		(property "Footprint" "Resistor_SMD:R_0603_1608Metric Resistor_SMD:R_0603_1608Metric"
+		(property "Footprint" "Resistor_SMD:R_0603_1608Metric Resistor_SMD_R_0603_1608Metric"
 			(at 106.172 43.18 90)
 			(hide yes)
@@
 			)
 		)
-		(property "Footprint" "Resistor_SMD:R_0603_1608Metric Resistor_SMD:R_0603_1608Metric"
+		(property "Footprint" "Resistor_SMD:R_0603_1608Metric Resistor_SMD_R_0603_1608Metric"
 			(at 254.762 85.09 90)
 			(hide yes)
@@
 			)
 		)
-		(property "Footprint" "Resistor_SMD:R_0603_1608Metric Resistor_SMD:R_0603_1608Metric"
+		(property "Footprint" "Resistor_SMD:R_0603_1608Metric Resistor_SMD_R_0603_1608Metric"
 			(at 256.032 125.73 90)
 			(hide yes)
@@
 			)
 		)
-		(property "Footprint" "Resistor_SMD:R_0603_1608Metric Resistor_SMD:R_0603_1608Metric"
+		(property "Footprint" "Resistor_SMD:R_0603_1608Metric Resistor_SMD_R_0603_1608Metric"
 			(at 264.287 162.56 90)
 			(hide yes)
