File: sub_interfaz.kicad_sch (KiCad schematic)
At the start: 29 parts, among them J13 Conn_01x11_Socket, J14 Conn_01x04_Socket, J15 Conn_01x04_Pin, J16 Conn_01x04_MountingPin, J17 Conn_01x04_Pin, SW4 SW_P, SW5 SW_P, SW6 SW_P, SW7 SW_P, SW8 SW_P, SW9 SW_P

Commit message: 10082026/B
nova revisão
Other:
- company: by todio -> ---
Changed lines of the file:
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@@
 	(title_block
 		(title "ihm i2sx3")
-		(date "2026-07-11")
-		(rev "0.1v")
-		(company "by todio")
-		(comment 1 "interface humano-maquina ")
+		(date "2026-08-10")
+		(rev "C")
+		(company "---")
+		(comment 1 "powered by STM32F407VET6")
+		(comment 2 "BY todio")
+		(comment 3 "na pagina \"hapia\" leia os aviosos e pergunta ")
 	)
 	(junction

Commit message: 10082026/D
"erros bobos"
Parts:
- removed R65: 100Ω, symbol Device:R
- added R91: 470Ω, symbol Device:R
- R68: value 100Ω -> 470Ω
Connections:
- net at D3.2 (A): now also R91.2
- net at J13.10 (Pin_10): now also R91.1
Changed lines of the file:
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@@
+	)
+	(symbol
+		(lib_id "Device:R")
+		(at 21.59 49.53 0)
+		(unit 1)
+		(body_style 1)
+		(exclude_from_sim no)
+		(in_bom yes)
+		(on_board yes)
+		(in_pos_files yes)
+		(dnp no)
+		(fields_autoplaced yes)
+		(property "Reference" "R91"
+			(at 24.13 48.2599 0)
+			(show_name no)
+			(do_not_autoplace no)
+			(effects
+				(font
+					(size 1.27 1.27)
+				)
+				(justify left)
+			)
+		)
+		(property "Value" "470Ω"
+			(at 24.13 50.7999 0)
+			(show_name no)
+			(do_not_autoplace no)
+			(effects
+				(font
+					(size 1.27 1.27)
+				)
+				(justify left)
+			)
+		)
+		(property "Footprint" ""
+			(at 19.812 49.53 90)
+			(hide yes)
+			(show_name no)
+			(do_not_autoplace no)
+			(effects
+				(font
+					(size 1.27 1.27)
+				)
+			)
+		)
+		(property "Datasheet" ""
+			(at 21.59 49.53 0)
+			(hide yes)
+			(show_name no)
+			(do_not_autoplace no)
+			(effects
+				(font
+					(size 1.27 1.27)
+				)
+			)
+		)
+		(property "Description" "Resistor"
+			(at 21.59 49.53 0)
+			(hide yes)
+			(show_name no)
+			(do_not_autoplace no)
+			(effects
+				(font
+					(size 1.27 1.27)
+				)
+			)
+		)
+		(pin "1"
+		)
+		(pin "2"
+		)
+		(instances
+			(project "hapia"
+				(path "/efba4993-d931-46ce-b72d-dcd9962acd35"
+					(reference "R91")
+					(unit 1)
+				)
+			)
+		)
 	)
 	(symbol
@@
 	)
 	(symbol
-		(lib_id "Device:R")
-		(at 21.59 49.53 0)
-		(unit 1)
-		(body_style 1)
-		(exclude_from_sim no)
-		(in_bom yes)
-		(on_board yes)
-		(in_pos_files yes)
-		(dnp no)
-		(property "Reference" "R65"
-			(at 24.13 48.2599 0)
-			(show_name no)
-			(do_not_autoplace no)
-			(effects
-				(font
-					(size 1.27 1.27)
-				)
-				(justify left)
-			)
-		)
-		(property "Value" "100Ω"
-			(at 24.13 50.8 0)
-			(show_name no)
-			(do_not_autoplace no)
-			(effects
-				(font
-					(size 1.27 1.27)
-				)
-				(justify left)
-			)
-		)
-		(property "Footprint" ""
-			(at 19.812 49.53 90)
-			(hide yes)
-			(show_name no)
-			(do_not_autoplace no)
-			(effects
-				(font
-					(size 1.27 1.27)
-				)
-			)
-		)
-		(property "Datasheet" ""
-			(at 21.59 49.53 0)
-			(hide yes)
-			(show_name no)
-			(do_not_autoplace no)
-			(effects
-				(font
-					(size 1.27 1.27)
-				)
-			)
-		)
-		(property "Description" "Resistor"
-			(at 21.59 49.53 0)
-			(hide yes)
-			(show_name no)
-			(do_not_autoplace no)
-			(effects
-				(font
-					(size 1.27 1.27)
-				)
-			)
-		)
-		(pin "1"
-		)
-		(pin "2"
-		)
-		(instances
-			(project "hapia"
-				(path "/efba4993-d931-46ce-b72d-dcd9962acd35"
-					(reference "R65")
-					(unit 1)
-				)
-			)
-		)
-	)
-	(symbol
 		(lib_id "power:GND")
 		(at 44.45 128.27 0)
@@
 			)
 		)
-		(property "Value" "100Ω"
+		(property "Value" "470Ω"
 			(at 43.18 50.7999 0)
 			(show_name no)

Commit message: 21082026/G
falta muita coisa
Parts:
- renumbered C83 to C87, C84 to C88, C85 to C89, C86 to C90, C87 to C91, C88 to C92, C89 to C93, C90 to C94, D3 to D5, D4 to D6, J13 to J14, J14 to J15, J15 to J16, J16 to J17, J17 to J18, R91 to R100, R66 to R101, R67 to R102, R68 to R103, R69 to R104, R70 to R105, R71 to R106, R72 to R107

Commit message: 29082026/I
Parts:
- C87, C88, C89, C90, C92, C93, C94: jlc_pcb: C346191 -> C307348; mouser: (none) -> 187-CL10B104KB8WPNC; mpn CL10B104KB8NFNC -> CL10B104KB8WPNC
Changed lines of the file:
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@@
 	(title_block
 		(title "ihm i2sx3")
-		(date "2026-08-10")
+		(date "2026-08-29")
 		(rev "C")
 		(company "---")
 		(comment 1 "powered by STM32F407VET6")
 		(comment 2 "BY todio")
-		(comment 3 "na pagina \"hapia\" leia os aviosos e pergunta ")
+		(comment 3 "na pagina \"hapia\" leia os avisos")
 	)
 	(junction
@@
 			)
 		)
-		(property "Datasheet" ""
+		(property "Datasheet" "https://www.lcsc.com/datasheet/C307348.pdf?spm=wm.sxq.inf.ggs___wm.fly.bg.0.xh&lcsc_vid=RFYLUFJeFgBYVgUARVEKU1ZUEwNcUQJQEVkIVlNSQgIxVlNeT1FfU1VRT1VYVDsOAxUeFF5JWBYZEEoKFBINSQcJGk4NBhADEA4cHktXRlVcSQwSGg0%3D"
 			(at 77.47 120.65 0)
 			(hide yes)
@@
 			)
 		)
-		(property "jlc_pcb:" "C346191"
+		(property "jlc_pcb:" "C307348"
+			(at 77.47 120.65 90)
+			(hide yes)
+			(show_name no)
+			(do_not_autoplace no)
+			(effects
+				(font
+					(size 1.27 1.27)
+				)
+			)
+		)
+		(property "mpn" "CL10B104KB8WPNC"
 			(at 77.47 120.65 90)
 			(hide yes)
@@
 			)
 		)
-		(property "mpn" "CL10B104KB8NFNC"
+		(property "mouser:" "187-CL10B104KB8WPNC"
 			(at 77.47 120.65 90)
 			(hide yes)
@@
 			)
 		)
-		(property "Datasheet" ""
+		(property "Datasheet" "https://www.lcsc.com/datasheet/C307348.pdf?spm=wm.sxq.inf.ggs___wm.fly.bg.0.xh&lcsc_vid=RFYLUFJeFgBYVgUARVEKU1ZUEwNcUQJQEVkIVlNSQgIxVlNeT1FfU1VRT1VYVDsOAxUeFF5JWBYZEEoKFBINSQcJGk4NBhADEA4cHktXRlVcSQwSGg0%3D"
 			(at 53.34 120.65 0)
 			(hide yes)
@@
 			)
 		)
-		(property "jlc_pcb:" "C346191"
+		(property "jlc_pcb:" "C307348"
 			(at 53.34 120.65 90)
 			(hide yes)
@@
 			)
 		)
-		(property "mpn" "CL10B104KB8NFNC"
+		(property "mpn" "CL10B104KB8WPNC"
+			(at 53.34 120.65 90)
+			(hide yes)
+			(show_name no)
+			(do_not_autoplace no)
+			(effects
+				(font
+					(size 1.27 1.27)
+				)
+			)
+		)
+		(property "mouser:" "187-CL10B104KB8WPNC"
 			(at 53.34 120.65 90)
 			(hide yes)
@@
 			)
 		)
-		(property "Datasheet" ""
+		(property "Datasheet" "https://www.lcsc.com/datasheet/C307348.pdf?spm=wm.sxq.inf.ggs___wm.fly.bg.0.xh&lcsc_vid=RFYLUFJeFgBYVgUARVEKU1ZUEwNcUQJQEVkIVlNSQgIxVlNeT1FfU1VRT1VYVDsOAxUeFF5JWBYZEEoKFBINSQcJGk4NBhADEA4cHktXRlVcSQwSGg0%3D"
 			(at 67.31 49.53 0)
 			(hide yes)
@@
 			)
 		)
-		(property "jlc_pcb:" "C346191"
+		(property "jlc_pcb:" "C307348"
 			(at 67.31 49.53 0)
 			(hide yes)
@@
 			)
 		)
-		(property "mpn" "CL10B104KB8NFNC"
+		(property "mpn" "CL10B104KB8WPNC"
+			(at 67.31 49.53 0)
+			(hide yes)
+			(show_name no)
+			(do_not_autoplace no)
+			(effects
+				(font
+					(size 1.27 1.27)
+				)
+			)
+		)
+		(property "mouser:" "187-CL10B104KB8WPNC"
 			(at 67.31 49.53 0)
 			(hide yes)
@@
 			)
 		)
-		(property "Datasheet" ""
+		(property "Datasheet" "https://www.lcsc.com/datasheet/C307348.pdf?spm=wm.sxq.inf.ggs___wm.fly.bg.0.xh&lcsc_vid=RFYLUFJeFgBYVgUARVEKU1ZUEwNcUQJQEVkIVlNSQgIxVlNeT1FfU1VRT1VYVDsOAxUeFF5JWBYZEEoKFBINSQcJGk4NBhADEA4cHktXRlVcSQwSGg0%3D"
 			(at 77.47 88.9 0)
 			(hide yes)
@@
 			)
 		)
-		(property "jlc_pcb:" "C346191"
+		(property "jlc_pcb:" "C307348"
 			(at 77.47 88.9 90)
 			(hide yes)
@@
 			)
 		)
-		(property "mpn" "CL10B104KB8NFNC"
+		(property "mpn" "CL10B104KB8WPNC"
+			(at 77.47 88.9 90)
+			(hide yes)
+			(show_name no)
+			(do_not_autoplace no)
+			(effects
+				(font
+					(size 1.27 1.27)
+				)
+			)
+		)
+		(property "mouser:" "187-CL10B104KB8WPNC"
 			(at 77.47 88.9 90)
 			(hide yes)
@@
 			)
 		)
-		(property "Datasheet" ""
+		(property "Datasheet" "https://www.lcsc.com/datasheet/C307348.pdf?spm=wm.sxq.inf.ggs___wm.fly.bg.0.xh&lcsc_vid=RFYLUFJeFgBYVgUARVEKU1ZUEwNcUQJQEVkIVlNSQgIxVlNeT1FfU1VRT1VYVDsOAxUeFF5JWBYZEEoKFBINSQcJGk4NBhADEA4cHktXRlVcSQwSGg0%3D"
 			(at 31.75 120.65 0)
 			(hide yes)
@@
 			)
 		)
-		(property "jlc_pcb:" "C346191"
+		(property "jlc_pcb:" "C307348"
 			(at 31.75 120.65 90)
 			(hide yes)
@@
 			)
 		)
-		(property "mpn" "CL10B104KB8NFNC"
+		(property "mpn" "CL10B104KB8WPNC"
+			(at 31.75 120.65 90)
+			(hide yes)
+			(show_name no)
+			(do_not_autoplace no)
+			(effects
+				(font
+					(size 1.27 1.27)
+				)
+			)
+		)
+		(property "mouser:" "187-CL10B104KB8WPNC"
 			(at 31.75 120.65 90)
 			(hide yes)
@@
 			)
 		)
-		(property "Datasheet" ""
+		(property "Datasheet" "https://www.lcsc.com/datasheet/C307348.pdf?spm=wm.sxq.inf.ggs___wm.fly.bg.0.xh&lcsc_vid=RFYLUFJeFgBYVgUARVEKU1ZUEwNcUQJQEVkIVlNSQgIxVlNeT1FfU1VRT1VYVDsOAxUeFF5JWBYZEEoKFBINSQcJGk4NBhADEA4cHktXRlVcSQwSGg0%3D"
 			(at 31.75 88.9 0)
 			(hide yes)
@@
 			)
 		)
-		(property "jlc_pcb:" "C346191"
+		(property "jlc_pcb:" "C307348"
+			(at 31.75 88.9 90)
+			(hide yes)
+			(show_name no)
+			(do_not_autoplace no)
+			(effects
+				(font
+					(size 1.27 1.27)
+				)
+			)
+		)
+		(property "mpn" "CL10B104KB8WPNC"
 			(at 31.75 88.9 90)
 			(hide yes)
@@
 			)
 		)
-		(property "mpn" "CL10B104KB8NFNC"
+		(property "mouser:" "187-CL10B104KB8WPNC"
 			(at 31.75 88.9 90)
 			(hide yes)
@@
 			)
 		)
-		(property "Datasheet" ""
+		(property "Datasheet" "https://www.lcsc.com/datasheet/C307348.pdf?spm=wm.sxq.inf.ggs___wm.fly.bg.0.xh&lcsc_vid=RFYLUFJeFgBYVgUARVEKU1ZUEwNcUQJQEVkIVlNSQgIxVlNeT1FfU1VRT1VYVDsOAxUeFF5JWBYZEEoKFBINSQcJGk4NBhADEA4cHktXRlVcSQwSGg0%3D"
 			(at 53.34 88.9 0)
 			(hide yes)
@@
 			)
 		)
-		(property "jlc_pcb:" "C346191"
+		(property "jlc_pcb:" "C307348"
+			(at 53.34 88.9 90)
+			(hide yes)
+			(show_name no)
+			(do_not_autoplace no)
+			(effects
+				(font
+					(size 1.27 1.27)
+				)
+			)
+		)
+		(property "mpn" "CL10B104KB8WPNC"
 			(at 53.34 88.9 90)
 			(hide yes)
@@
 			)
 		)
-		(property "mpn" "CL10B104KB8NFNC"
+		(property "mouser:" "187-CL10B104KB8WPNC"
 			(at 53.34 88.9 90)
 			(hide yes)

Commit message: o .bom não foi terminado
O desafio e todo custar menos de 150 dólares(eua) e menos de 1000r(reais)
Parts:
- removed C87, C88, C89, C90: 100nf, Capacitor_SMD:C_0603_1608Metric, symbol Device:C
- added CN4: 100nf, Capacitor_SMD:C_0603_1608Metric, symbol Device:C_Network04
- C91: footprint (none) -> Capacitor_SMD:C_1206_3216Metric_Pad1.33x1.80mm_HandSolder; jlc_pcb: (none) -> C13585; mouser: (none) -> 187-CL31B106KLK6PNE; mpn (none) -> CL31A106KBHNNNE
- J16, J18: footprint (none) -> Connector_JST:JST_EH_B4B-EH-A_1x04_P2.50mm_Vertical
- SW4, SW5, SW6, SW7, SW8, SW9: footprint (none) -> Button_Switch_THT:SW_PUSH_6mm_H5mm; jlc_pcb: (none) -> C139756; mouser: (none) -> 688-SKHHAM; mpn (none) -> SKHHAMA010
Connections:
- net GND: now also CN4.5 (C4), CN4.6 (C3), CN4.7 (C2), CN4.8 (C1)
- net S_1: now also CN4.1 (common)
- net S_2: now also CN4.2 (C1)
- net S_4: now also CN4.3 (C2)
- net S_5: now also CN4.4 (C3)

Commit message: 27092026/0002
Parts:
- D5, D6: value LED -> RED; footprint (none) -> LED_THT:LED_D3.0mm_FlatTop; jlc_pcb: (none) -> C7148823; mouser: (none) -> 78-VLCS5130; mpn (none) -> VLCS5130
- R100, R103: footprint (none) -> Resistor_SMD:R_0805_2012Metric_Pad1.20x1.40mm_HandSolder; jlc_pcb: (none) -> C114564; mouser: (none) -> 603-RC0805FR-07470RL; mpn (none) -> RC0805FR-07470RL
- R101, R102, R104, R105, R106: footprint (none) -> Capacitor_SMD:C_0603_1608Metric_Pad1.08x0.95mm_HandSolder; jlc_pcb: (none) -> C22548; mouser: (none) -> 603-RC0603FR-071KL; mpn (none) -> RC0603FR-071KL
- R107: footprint (none) -> Capacitor_SMD:C_0603_1608Metric_Pad1.08x0.95mm_HandSolder; jlc_pcb: (none) -> C22548; mouser: (none) -> 603-RC0603FR-071KL; mpn (none) -> RC0603FR-071KL; now not fitted
